Commit message: Rename LSR200Auto Lite ROS package to AKM naming

File: platforms/lucsys_lsr200auto_akm_lite_description/urdf/lsr200auto_akm_lite.urdf (robot description, URDF)
Before this commit: robot lucsys_lsr200auto_ackermann_lite, 9 links, 8 joints
Links:
- link base_link: geometry collision mesh filename=package://lucsys_lsr200auto_akm_lite_description/meshes/lsr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; visual mesh filename=package://lucsys_lsr200auto_akm_lite_description/meshes/lsr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
- link camera_link: geometry collision mesh filename=package://lucsys_lsr200auto_akm_lite_description/meshes/lsr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; visual mesh filename=package://lucsys_lsr200auto_akm_lite_description/meshes/lsr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
- link gyro_link: geometry collision mesh filename=package://lucsys_lsr200auto_akm_lite_description/meshes/lsr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; visual mesh filename=package://lucsys_lsr200auto_akm_lite_description/meshes/lsr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
- link laser_link: geometry collision mesh filename=package://lucsys_lsr200auto_akm_lite_description/meshes/lsr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; visual mesh filename=package://lucsys_lsr200auto_akm_lite_description/meshes/lsr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
- link lb_wheel_link: geometry collision mesh filename=package://lucsys_lsr200auto_akm_lite_description/meshes/lsr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; visual mesh filename=package://lucsys_lsr200auto_akm_lite_description/meshes/lsr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
- link lf_wheel_link: geometry collision mesh filename=package://lucsys_lsr200auto_akm_lite_description/meshes/lsr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; visual mesh filename=package://lucsys_lsr200auto_akm_lite_description/meshes/lsr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
- link rb_wheel_link: geometry collision mesh filename=package://lucsys_lsr200auto_akm_lite_description/meshes/lsr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; visual mesh filename=package://lucsys_lsr200auto_akm_lite_description/meshes/lsr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
- link rf_wheel_link: geometry collision mesh filename=package://lucsys_lsr200auto_akm_lite_description/meshes/lsr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; visual mesh filename=package://lucsys_lsr200auto_akm_lite_description/meshes/lsr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
- link rtk_link: geometry collision mesh filename=package://lucsys_lsr200auto_akm_lite_description/meshes/lsr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; visual mesh filename=package://lucsys_lsr200auto_akm_lite_description/meshes/lsr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
